Commit message: map -> odom tf not being published (idk why)

File: description/lidar.xacro (robot description, xacro)
@@ -21,5 +21,5 @@
 </link>
 <joint name="lidar_joint" type="fixed">
-  <parent link="chassis"/>
+  <parent link="base_link"/>
   <child link="lidar_link"/>
   <origin xyz="0 0 0.13" rpy="0 0 0"/>

Commit message: add ros2_control e  twist_mux (ainda não está sub de /cmd_vel)

File: description/lidar.xacro (robot description, xacro)
@@ -1,5 +1,5 @@
 <?xml version="1.0"?>
 <robot xmlns:xacro="http://www.ros.org/wiki/xacro" >
-<link name="lidar_link">
+<link name="laser_link">
   <inertial>
     <origin xyz="0 0 0" rpy="0 0 0"/>
@@ -22,8 +22,8 @@
 <joint name="lidar_joint" type="fixed">
   <parent link="base_link"/>
-  <child link="lidar_link"/>
+  <child link="laser_link"/>
   <origin xyz="0 0 0.13" rpy="0 0 0"/>
 </joint>
-<gazebo reference="lidar_link">
+<gazebo reference="laser_link">
   <sensor name="lidar" type="ray">
     <pose>0 0 0 0 0 0</pose>
@@ -53,8 +53,8 @@
     <plugin name="scan" filename="libgazebo_ros_ray_sensor.so">
       <ros>
-        <argument>--ros-args --remap ~/out:=scan</argument>
+        <argument>~/out:=scan</argument>
       </ros>
       <output_type>sensor_msgs/LaserScan</output_type>
-      <frame_name>lidar_link</frame_name>
+      <frame_name>laser_link</frame_name>
     </plugin>
   </sensor>

File: description/robot.urdf.xacro (robot description, xacro)
@@ -1,7 +1,12 @@
 <?xml version="1.0"?>
 <robot xmlns:xacro="http://www.ros.org/wiki/xacro"  name="robot">
-	<!--<xacro:include filename="robot_core_lr.xacro"/>-->
-	<xacro:include filename="robot_core_lr.xacro"/>
-	<xacro:include filename="gazebo_control.xacro"/>
-	<xacro:include filename="lidar.xacro"/>
+    <xacro:arg name="use_ros2_control" default="true"/>
+    <xacro:include filename="robot_core_lr.xacro" />
+    <xacro:if value="$(arg use_ros2_control)">
+        <xacro:include filename="ros2_control.xacro" />
+    </xacro:if>
+    <xacro:unless value="$(arg use_ros2_control)">
+        <xacro:include filename="gazebo_control.xacro" />
+    </xacro:unless>
+    <xacro:include filename="lidar.xacro" />
 </robot>
